File: kicad-cassandra/can.kicad_sch (KiCad schematic)
At the start: 11 parts, among them J3 DE9_Pins_MountingHoles, SW4 SW_SPDT, U3 SN65HVD232

Commit message: add wire only possibility
Parts:
- added J7: ~, cassandra:CONN4_05010302_WRE, symbol cassandra:691401700002B
Connections:
- net CAN_HIGH: now also J7.1, J7.A1 (1)
- net CAN_LOW: now also J7.2, J7.A2 (2)
