File: kicad-cassandra/kicad-cassandra.kicad_sch (KiCad schematic)
At the start: 29 parts, among them J1 Conn_ST_STDC14, SW1 SW_Push, SW2 SW_Push, SW3 SW_Push, U2 STM32F446RETx, Y1 831024589

Commit message: make sure usb works
Connections:
- net HOST_VCP_RX: now also U2.43 (PA10); no longer U2.42 (PA9)
- net HOST_VCP_TX: now also U2.42 (PA9); no longer U2.43 (PA10)
- net TGT_VCP_RX: now also U2.17 (PA3); no longer U2.16 (PA2)
- net TGT_VCP_TX: now also U2.16 (PA2); no longer U2.17 (PA3)
Changed lines of the file:
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@@
 		)
 	)
-	(label "TGT_VCP_TX"
+	(label "TGT_VCP_RX"
 		(at 139.7 43.18 0)
 		(effects
@@
 		)
 	)
-	(label "HOST_VCP_RX"
-		(at 139.7 58.42 0)
+	(label "TGT_VCP_TX"
+		(at 139.7 40.64 0)
 		(effects
 			(font
@@
 		)
 	)
+	(label "HOST_VCP_RX"
+		(at 139.7 60.96 0)
+		(effects
+			(font
+				(size 1.27 1.27)
+			)
+			(justify left bottom)
+		)
+	)
 	(label "TGT_VCP_RX"
 		(at 59.69 158.75 0)
@@
 		)
 	)
-	(label "HOST_VCP_TX"
-		(at 139.7 60.96 0)
-		(effects
-			(font
-				(size 1.27 1.27)
-			)
-			(justify left bottom)
-		)
-	)
 	(label "TGT_SWDIO"
 		(at 59.69 151.13 0)
@@
 		)
 	)
-	(label "TGT_VCP_RX"
-		(at 139.7 40.64 0)
-		(effects
-			(font
-				(size 1.27 1.27)
-			)
-			(justify left bottom)
-		)
-	)
 	(label "uSD_CLK"
 		(at 190.5 82.55 180)
@@
 		)
 	)
+	(label "HOST_VCP_TX"
+		(at 139.7 58.42 0)
+		(effects
+			(font
+				(size 1.27 1.27)
+			)
+			(justify left bottom)
+		)
+	)

Commit message: add wire only possibility
Parts:
- removed D3, D4, D5, D6: AMBER, cassandra:WL-SMSW_0603_ROUND, symbol Device:LED
- removed R4, R5, R6, R7: 230, Resistor_SMD:R_0603_1608Metric, symbol Device:R_Small
- D1, D2: footprint cassandra:WL-SMSW_0603_ROUND -> LED_SMD:LED_0603_1608Metric_Pad1.05x0.95mm_HandSolder
Connections:
- net LED_BIT0: no longer names the net of U2.4 (PC15)
- net LED_BIT1: no longer names the net of U2.3 (PC14)
- net LED_BIT2: no longer names the net of U2.2 (PC13)
- net LED_BIT3: no longer names the net of U2.62 (PB9)
- net USB_CC1_READ: no longer names the net of U2.9 (PC1)
- net USB_CC2_READ: no longer names the net of U2.8 (PC0)
- no-connect marks 15 -> 21
Other:
- sheet USB ports: added none; removed USB_CC1_READ, USB_CC2_READ
